File: projects/TestBoard/Combine-CPU-POWER-RELAY-smd.brd (EAGLE design)
At the start: 88.1 x 54.4 mm, 34 parts

Commit message: 14-8-59
Routing:
- net 3V3: track 160.3 -> 166.5 mm
- net +5V: track 185.0 -> 186.9 mm
Other:
- board text added: "Tong"
