File: projects/IoT/test2.sch (EAGLE design)
At the start: 3 parts

Commit message: r61
Parts:
- removed JP1: (no value), pinhead:PINHD-2X11/90
- removed U3: (no value), esp8266modules:ESP12ESMD
- added U$1: HLK-PM01, HLK-PM01:HLK-PM01
- added U$2: FEMALE-PLUG, Male-Female-PLUG:FEMALE-PLUG
- added U$3: MALE-PLUG, Male-Female-PLUG:MALE-PLUG
- added U$4: POWER-RELAY-FOOTPRINT, Power-Plug-Footprint:POWER-RELAY-FOOTPRINT
- added U$5: TACT-SWITCH-SMD, Tact-Switch-SMD:TACT-SWITCH-SMD
- added U$6: FUSE-CLIP, Fuse-Clip:FUSE-CLIP
Changed lines of the file:
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@@
 <?xml version="1.0" encoding="utf-8"?>
 <!DOCTYPE eagle SYSTEM "eagle.dtd">
-<eagle version="7.5.0">
+<eagle version="7.6.0">
 <drawing>
 <settings>
@@
 <setting verticaltext="up"/>
 </settings>
-<grid distance="10" unitdist="mil" unit="mil" style="lines" multiple="1" display="no" altdistance="25" altunitdist="mil" altunit="mil"/>
+<grid distance="0.1" unitdist="inch" unit="inch" style="lines" multiple="1" display="no" altdistance="0.01" altunitdist="inch" altunit="inch"/>
 <layers>
 <layer number="1" name="Top" color="4" fill="1" visible="no" active="no"/>
@@
 <parts>
 <part name="FRAME1" library="SparkFun-Aesthetics" deviceset="FRAME-LEDGER" device=""/>
-<part name="JP1" library="pinhead" deviceset="PINHD-2X11" device="/90"/>
-<part name="U3" library="esp8266modules" deviceset="ESP12E" device="SMD"/>
+<part name="U$1" library="HLK-PM01" deviceset="HLK-PM01" device=""/>
+<part name="U$2" library="Male-Female-PLUG" deviceset="FEMALE-PLUG" device=""/>
+<part name="U$3" library="Male-Female-PLUG" deviceset="MALE-PLUG" device=""/>
+<part name="U$4" library="Power-Plug-Footprint" deviceset="POWER-RELAY-FOOTPRINT" device=""/>
+<part name="U$5" library="Tact-Switch-SMD" deviceset="TACT-SWITCH-SMD" device=""/>
+<part name="U$6" library="Fuse-Clip" deviceset="FUSE-CLIP" device=""/>
 </parts>
 <sheets>
@@
 <instance part="FRAME1" gate="G$1" x="-15.24" y="40.64"/>
 <instance part="FRAME1" gate="G$2" x="314.96" y="40.64"/>
-<instance part="JP1" gate="A" x="48.26" y="195.58"/>
-<instance part="U3" gate="G$1" x="93.98" y="208.28"/>
+<instance part="U$1" gate="G$1" x="33.02" y="284.48"/>
+<instance part="U$2" gate="G$1" x="35.56" y="248.92"/>
+<instance part="U$3" gate="G$1" x="33.02" y="218.44"/>
+<instance part="U$4" gate="G$1" x="38.1" y="190.5"/>
+<instance part="U$5" gate="G$1" x="30.48" y="162.56"/>
+<instance part="U$6" gate="1" x="30.48" y="154.94"/>
 </instances>
 <busses>
@@
 </schematic>
 </drawing>
-<compatibility>
-<note version="6.3" minversion="6.2.2" severity="warning">
-Since Version 6.2.2 text objects can contain more than one line,
-which will not be processed correctly with this version.
-</note>
-</compatibility>
 </eagle>
