File: projects/PlugV1/Plugv1.brd (EAGLE design)
At the start: 100 x 80 mm, 7 parts

Commit message: r61
Parts:
- removed FRAME1: FRAME-LEDGER, SparkFun-Aesthetics:CREATIVE_COMMONS
- removed U$3: MALE-PLUG, Male-Female-PLUG:MALE-PLUG
- removed U$4: POWER-RELAY-FOOTPRINT, Power-Plug-Footprint:POWER-RELAY-FOOTPRINT
- removed U$5: TACT-SWITCH-SMD, Tact-Switch-SMD:TACT-SWITCH-SMD
- removed U$6: FUSE-CLIP, Fuse-Clip:FUSE-CLIP
- added F1: (no value), fuse:SH22,5A
- added X1: (no value), con-ptr500:AK500/2-H
- U$2: value FEMALE-PLUG -> REG-AMS1117-3.3V; device Male-Female-PLUG:FEMALE-PLUG -> diy-modules:REG-AMS1117
- moved U$2 162.9 mm to (42.8, 22.3), turned to 270 degrees
- moved U$1 109.1 mm to (0.81, 12.5)
Connections:
- new net N$1: U$1.P$4, U$2.J1.2
- new net N$2: U$1.P$3, U$2.J1.1
- new net N$3: F1.2, U$1.P$1
- new net N$4: F1.1, X1.1
- new net N$5: U$1.P$2, X1.2
Routing:
- net N$22: track 29.8 -> 0.00 mm
- net N$13: track 26.2 -> 0.00 mm
- net N$14: track 25.7 -> 0.00 mm
- net N$20: track 25.0 -> 0.00 mm
- net N$21: track 24.6 -> 0.00 mm
- net N$11: track 22.1 -> 0.00 mm
- net N$12: track 21.0 -> 0.00 mm
- net N$19: track 19.6 -> 0.00 mm
- net N$18: track 19.6 -> 0.00 mm
- net N$9: track 17.3 -> 0.00 mm
- net N$10: track 16.6 -> 0.00 mm
- net N$16: track 14.8 -> 0.00 mm
- net N$17: track 14.3 -> 0.00 mm
- net N$7: track 12.6 -> 0.00 mm
- net N$8: track 12.1 -> 0.00 mm
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