File: projects/SmartPlugV3/plug-v24-Make-board-myself-to-test-circuit.brd (EAGLE design)
At the start: 63.5 x 70 mm, 34 parts

Commit message: commit message
Parts:
- removed CIN1/TAN, COUT1/TAN: 22uF, rcl:B/3528-21R
- added CT1: 47UF, Seeed-OPL-Capacitor:ELECTRO-SMD-C-6MM
- moved U$1 16.5 mm to (30.2, 56.2), turned to 180 degrees
- moved C2 11.0 mm to (48.4, 27.3), turned to 0 degrees
- moved V1 6.92 mm to (35.5, 66.4), turned to 270 degrees
- moved TR 5.63 mm to (41.6, 29.1)
- moved X1 5.30 mm to (49.0, 58.5)
- moved LED-RELAY 5.22 mm to (54.0, 14.8)
- moved LED-NET 5.21 mm to (54.0, 12.0)
- moved LED-ESP 5.20 mm to (54.0, 9.05)
- moved EXT 5.17 mm to (53.0, 19.4)
- moved X2 5.03 mm to (11.4, 58.5)
- moved R-NET 4.21 mm to (43.6, 11.4)
- moved R-TR 4.16 mm to (37.4, 30.2)
- moved COUT2/CE 4.16 mm to (20.9, 45.1), turned to 180 degrees
- moved R-OPTO 1.55 mm to (32.3, 21.2)
- moved REG 1.45 mm to (13.1, 42.0)
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Connections:
- net +5V: no longer CIN1/TAN.+
- net 3V3: now also CT1.+; no longer COUT1/TAN.+
- net GND: now also CT1.-; no longer CIN1/TAN.-, COUT1/TAN.-
Routing:
- net N: track 68.3 -> 98.2 mm
- net RELAY-COM: track 88.9 -> 64.8 mm
- net GND: track 244.1 -> 230.2 mm
- net +5V: track 121.5 -> 107.7 mm
- net RELAY-NO: track 58.1 -> 47.8 mm
- net G-12: track 60.8 -> 54.1 mm
- net G-13: track 50.8 -> 44.8 mm
- net N$21: track 20.2 -> 14.8 mm
- net N$6: track 28.6 -> 23.3 mm
- net N$17: track 42.7 -> 47.5 mm
- net G-14: track 39.2 -> 34.4 mm
- net 3V3: track 105.4 -> 108.2 mm
- net N$1: track 6.20 -> 7.75 mm
- net N$2: track 3.82 -> 2.33 mm
- net N$13: track 4.83 -> 6.08 mm
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Other:
- board size 63.5 x 70 mm -> 59 x 70 mm
- board text added: "Tong"
